File: hardware/sfy/sfy.kicad_pcb (KiCad board)
At the start: 2 copper layers, 80.3 x 80.3 mm, 0 parts

Commit message: add led
Routing:
- net (no net): track 0.00 -> 26.0 mm, vias 0 -> 2
Changed lines of the file:
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@@
   (net 0 "")
   (gr_circle (center 149.86 91.44) (end 172.72 124.46) (layer "Edge.Cuts") (width 0.1) (fill none))
+  (segment (start 175.26 81.28) (end 170.18 76.2) (width 0.2) (layer "F.Cu") (net 0))
+  (segment (start 175.26 86.36) (end 175.26 81.28) (width 0.2) (layer "F.Cu") (net 0))
+  (segment (start 167.64 78.74) (end 167.64 88.9) (width 0.2) (layer "F.Cu") (net 0))
+  (segment (start 170.18 76.2) (end 167.64 78.74) (width 0.2) (layer "F.Cu") (net 0))
+  (via (at 175.26 86.36) (size 0.8) (drill 0.4) (layers "F.Cu" "B.Cu") (free) (net 0))
+  (via (at 167.64 88.9) (size 0.8) (drill 0.4) (layers "F.Cu" "B.Cu") (free) (net 0))
 )
